File: docs/MHS_Mobile_Hardware_Sampler_V3/MHS_Mobile_Hardware_Sampler_V3.kicad_pcb (KiCad board)
At the start: 2 copper layers, 198 x 143.5 mm, 48 parts, among them J1 Conn_01x14_MountingPin, J10 Conn_01x02, J11 NMJ4HCD2, J16 NMJ4HCD2, J17 NMJ4HCD2, J18 NMJ4HCD2, J2 Conn_01x14_MountingPin, J3 DIN-5, J4 06JQ-BT, J5 Conn_01x07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

Commit message: Updated Kicad Project
Parts:
- R1, R2, R3, R4, R5, R6, R7, R8: footprint Resistor_THT:R_Axial_DIN0411_L9.9mm_D3.6mm_P7.62mm_Vertical -> Resistor_THT:R_Axial_DIN0411_L9.9mm_D3.6mm_P12.70mm_Horizontal
- moved J?3=FSR4;6=FSR1 44.7 mm to (150.5, 156.0)
- moved R1 7.86 mm to (204.0, 118.7)
- moved R2 7.86 mm to (210.5, 118.7)
- moved H11 7.40 mm to (73.4, 115.5)
- moved H12 7.40 mm to (112.0, 115.6)
- moved H13 7.40 mm to (151.0, 115.6)
- moved H14 7.40 mm to (190.0, 115.1)
- moved H5V1 7.40 mm to (53.5, 115.5)
- moved H5V3 7.40 mm to (131.0, 115.6)
- moved H5V4 7.40 mm to (170.0, 115.1)
- moved H5V2 7.40 mm to (92.0, 115.7)
- moved R7 6.91 mm to (188.0, 75.8)
- moved R6 5.50 mm to (161.0, 74.0)
- moved R5 4.83 mm to (155.5, 50.1)
- moved R3 2.88 mm to (204.0, 136.2)
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Routing:
- net Net-(H13-Pad1): track 92.0 -> 133.1 mm, vias 3 -> 2
- net Net-(H11-Pad1): track 250.0 -> 209.8 mm
- net Net-(H5V1-Pad1): track 206.5 -> 237.6 mm
- net Net-(J?3=FSR4;6=FSR1-Pad1): track 91.6 -> 119.2 mm, vias 0 -> 1
- net Net-(H12-Pad1): track 146.1 -> 130.6 mm, vias 1 -> 2
- net Net-(J8-Pad4): track 44.0 -> 30.0 mm
- net Net-(J10-Pad1): track 73.3 -> 85.5 mm
- net Net-(J2-Pad12): track 227.5 -> 237.3 mm
- net Net-(H14-Pad1): track 98.9 -> 107.3 mm, vias 1 -> 0
- net Net-(C1-Pad1): track 247.3 -> 239.1 mm
- net Net-(J3-Pad4): track 24.9 -> 20.1 mm
