File: docs/MHS_Mobile_Hardware_Sampler_V3/MHS_Mobile_Hardware_Sampler_V3.kicad_sch (KiCad schematic)
At the start: 48 parts, among them J1 Conn_01x14_MountingPin, J10 Conn_01x02, J11 NMJ4HCD2, J16 NMJ4HCD2, J17 NMJ4HCD2, J18 NMJ4HCD2, J2 Conn_01x14_MountingPin, J3 DIN-5, J4 06JQ-BT, J5 Conn_01x07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

Commit message: Updated Kicad Project
Parts:
- R1, R2, R3, R4, R5, R6, R7, R8: footprint Resistor_THT:R_Axial_DIN0411_L9.9mm_D3.6mm_P7.62mm_Vertical -> (none)
Changed lines of the file:
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@@
       (effects (font (size 1.27 1.27)) (justify left))
     )
-    (property "Footprint" "Resistor_THT:R_Axial_DIN0411_L9.9mm_D3.6mm_P7.62mm_Vertical" (id 2) (at 126.492 160.02 90)
+    (property "Footprint" "" (id 2) (at 126.492 160.02 90)
       (effects (font (size 1.27 1.27)) hide)
     )
@@
       (effects (font (size 1.27 1.27)) (justify left))
     )
-    (property "Footprint" "Resistor_THT:R_Axial_DIN0411_L9.9mm_D3.6mm_P7.62mm_Vertical" (id 2) (at 375.412 31.75 90)
+    (property "Footprint" "" (id 2) (at 375.412 31.75 90)
       (effects (font (size 1.27 1.27)) hide)
     )
@@
       (effects (font (size 1.27 1.27)) (justify left))
     )
-    (property "Footprint" "Resistor_THT:R_Axial_DIN0411_L9.9mm_D3.6mm_P7.62mm_Vertical" (id 2) (at 126.492 181.61 90)
+    (property "Footprint" "" (id 2) (at 126.492 181.61 90)
       (effects (font (size 1.27 1.27)) hide)
     )
@@
     (property "Reference" "R5" (id 0) (at 325.12 20.32 90))
     (property "Value" "R220" (id 1) (at 325.12 22.86 90))
-    (property "Footprint" "Resistor_THT:R_Axial_DIN0411_L9.9mm_D3.6mm_P7.62mm_Vertical" (id 2) (at 325.12 28.448 90)
+    (property "Footprint" "" (id 2) (at 325.12 28.448 90)
       (effects (font (size 1.27 1.27)) hide)
     )
@@
       (effects (font (size 1.27 1.27)) (justify left))
     )
-    (property "Footprint" "Resistor_THT:R_Axial_DIN0411_L9.9mm_D3.6mm_P7.62mm_Vertical" (id 2) (at 395.732 64.77 90)
+    (property "Footprint" "" (id 2) (at 395.732 64.77 90)
       (effects (font (size 1.27 1.27)) hide)
     )
@@
       (effects (font (size 1.27 1.27)) (justify left))
     )
-    (property "Footprint" "Resistor_THT:R_Axial_DIN0411_L9.9mm_D3.6mm_P7.62mm_Vertical" (id 2) (at 394.462 30.48 90)
+    (property "Footprint" "" (id 2) (at 394.462 30.48 90)
       (effects (font (size 1.27 1.27)) hide)
     )
@@
       (effects (font (size 1.27 1.27)) (justify left))
     )
-    (property "Footprint" "Resistor_THT:R_Axial_DIN0411_L9.9mm_D3.6mm_P7.62mm_Vertical" (id 2) (at 50.292 180.34 90)
+    (property "Footprint" "" (id 2) (at 50.292 180.34 90)
       (effects (font (size 1.27 1.27)) hide)
     )
@@
       (effects (font (size 1.27 1.27)) (justify left))
     )
-    (property "Footprint" "Resistor_THT:R_Axial_DIN0411_L9.9mm_D3.6mm_P7.62mm_Vertical" (id 2) (at 52.832 147.32 90)
+    (property "Footprint" "" (id 2) (at 52.832 147.32 90)
       (effects (font (size 1.27 1.27)) hide)
     )
@@
     )
     (path "/c2f40f12-9140-473b-8e1d-752c1c930d8b"
-      (reference "R1") (unit 1) (value "R_Variable") (footprint "Resistor_THT:R_Axial_DIN0411_L9.9mm_D3.6mm_P7.62mm_Vertical")
+      (reference "R1") (unit 1) (value "R_Variable") (footprint "Resistor_THT:R_Axial_DIN0411_L9.9mm_D3.6mm_P12.70mm_Horizontal")
     )
     (path "/ebdccc38-546b-4d29-8a1d-1ab8adf77e08"
-      (reference "R2") (unit 1) (value "R_Variable") (footprint "Resistor_THT:R_Axial_DIN0411_L9.9mm_D3.6mm_P7.62mm_Vertical")
+      (reference "R2") (unit 1) (value "R_Variable") (footprint "Resistor_THT:R_Axial_DIN0411_L9.9mm_D3.6mm_P12.70mm_Horizontal")
     )
     (path "/0e6aea34-c909-43eb-ab34-679ff8f629ea"
-      (reference "R3") (unit 1) (value "R_Variable") (footprint "Resistor_THT:R_Axial_DIN0411_L9.9mm_D3.6mm_P7.62mm_Vertical")
+      (reference "R3") (unit 1) (value "R_Variable") (footprint "Resistor_THT:R_Axial_DIN0411_L9.9mm_D3.6mm_P12.70mm_Horizontal")
     )
     (path "/3a878acd-db72-4060-9445-ca901d7fd684"
-      (reference "R4") (unit 1) (value "R_Variable") (footprint "Resistor_THT:R_Axial_DIN0411_L9.9mm_D3.6mm_P7.62mm_Vertical")
+      (reference "R4") (unit 1) (value "R_Variable") (footprint "Resistor_THT:R_Axial_DIN0411_L9.9mm_D3.6mm_P12.70mm_Horizontal")
     )
     (path "/4ed70811-c8d4-4de3-9055-2b61827964a3"
-      (reference "R5") (unit 1) (value "R220") (footprint "Resistor_THT:R_Axial_DIN0411_L9.9mm_D3.6mm_P7.62mm_Vertical")
+      (reference "R5") (unit 1) (value "R220") (footprint "Resistor_THT:R_Axial_DIN0411_L9.9mm_D3.6mm_P12.70mm_Horizontal")
     )
     (path "/275c3e87-6b92-4445-ae44-835199568f46"
-      (reference "R6") (unit 1) (value "R470") (footprint "Resistor_THT:R_Axial_DIN0411_L9.9mm_D3.6mm_P7.62mm_Vertical")
+      (reference "R6") (unit 1) (value "R470") (footprint "Resistor_THT:R_Axial_DIN0411_L9.9mm_D3.6mm_P12.70mm_Horizontal")
     )
     (path "/a55421f9-e4b3-4b95-9a5c-a833b0f7321f"
-      (reference "R7") (unit 1) (value "R47") (footprint "Resistor_THT:R_Axial_DIN0411_L9.9mm_D3.6mm_P7.62mm_Vertical")
+      (reference "R7") (unit 1) (value "R47") (footprint "Resistor_THT:R_Axial_DIN0411_L9.9mm_D3.6mm_P12.70mm_Horizontal")
     )
     (path "/8a532a5e-bef9-4902-a8e4-8351de1e5086"
-      (reference "R8") (unit 1) (value "R47") (footprint "Resistor_THT:R_Axial_DIN0411_L9.9mm_D3.6mm_P7.62mm_Vertical")
+      (reference "R8") (unit 1) (value "R47") (footprint "Resistor_THT:R_Axial_DIN0411_L9.9mm_D3.6mm_P12.70mm_Horizontal")
     )
     (path "/968876f6-82e7-4e81-aa4a-d5e5e11ed1a1"
