File: docs/KiCad/Lunchbox_Sampler_FSR_PCB/Lunchbox_Sampler_FSR_PCB.kicad_pcb (KiCad board)
At the start: 2 copper layers, 185.3 x 55 mm, 19 parts

Commit message: pcb updated
Routing:
- net Net-(H11-Pad1): track 215.7 -> 206.6 mm
- net Net-(H12-Pad1): track 130.4 -> 124.4 mm
Changed lines of the file:
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@@
       (effects (font (size 1 1) (thickness 0.15)))
     )
-    (fp_text value "MountingHole_Pad" (at -44.9 -4.75) (layer "F.Fab")
+    (fp_text value "MountingHole_Pad" (at 0.1 -26.5) (layer "F.Fab")
       (effects (font (size 1 1) (thickness 0.15)))
     )
@@
   (gr_rect (start 86 119) (end 118 151) (layer "User.4") (width 0.15) (fill none))
   (gr_rect (start 47 119) (end 79 151) (layer "User.4") (width 0.15) (fill none))
-  (segment (start 73.5 115.6) (end 73.5 137.4) (width 1) (layer "F.Cu") (net 1))
+  (segment (start 73.5 129.38) (end 73.5 115.6) (width 1) (layer "F.Cu") (net 1))
   (segment (start 171.32 151) (end 166.32 156) (width 1) (layer "F.Cu") (net 1))
-  (segment (start 73.5 137.5) (end 73.4 137.6) (width 1) (layer "F.Cu") (net 1))
+  (segment (start 81.28 137.16) (end 73.5 129.38) (width 1) (layer "F.Cu") (net 1))
   (segment (start 166.32 156) (end 163 156) (width 1) (layer "F.Cu") (net 1))
   (via (at 171.32 151) (size 2) (drill 0.4) (layers "F.Cu" "B.Cu") (net 1))
-  (via (at 73.5 137.4) (size 2) (drill 0.4) (layers "F.Cu" "B.Cu") (net 1))
-  (segment (start 123.229966 145.729966) (end 74.609966 145.729966) (width 1) (layer "B.Cu") (net 1))
+  (via (at 81.28 137.16) (size 2) (drill 0.4) (layers "F.Cu" "B.Cu") (net 1))
+  (segment (start 128.5 151) (end 163 151) (width 1) (layer "B.Cu") (net 1))
   (segment (start 215.9 151.6) (end 215.9 135.4) (width 1) (layer "B.Cu") (net 1))
-  (segment (start 73.5 144.62) (end 74.609966 145.729966) (width 1) (layer "B.Cu") (net 1))
   (segment (start 208 159.5) (end 215.9 151.6) (width 1) (layer "B.Cu") (net 1))
+  (segment (start 89.849966 145.729966) (end 123.229966 145.729966) (width 1) (layer "B.Cu") (net 1))
   (segment (start 163 151) (end 164 151) (width 1) (layer "B.Cu") (net 1))
   (segment (start 171.32 151) (end 174 151) (width 1) (layer "B.Cu") (net 1))
-  (segment (start 73.5 137.4) (end 73.5 144.62) (width 1) (layer "B.Cu") (net 1))
   (segment (start 163 151) (end 171.32 151) (width 1) (layer "B.Cu") (net 1))
-  (segment (start 163 151) (end 128.5 151) (width 1) (layer "B.Cu") (net 1))
+  (segment (start 123.229966 145.729966) (end 128.5 151) (width 1) (layer "B.Cu") (net 1))
   (segment (start 174 151) (end 182.5 159.5) (width 1) (layer "B.Cu") (net 1))
   (segment (start 211.85 131.35) (end 210.5 131.35) (width 1) (layer "B.Cu") (net 1))
-  (segment (start 128.5 151) (end 123.229966 145.729966) (width 1) (layer "B.Cu") (net 1))
   (segment (start 182.5 159.5) (end 208 159.5) (width 1) (layer "B.Cu") (net 1))
   (segment (start 215.9 135.4) (end 211.85 131.35) (width 1) (layer "B.Cu") (net 1))
-  (segment (start 112 115.6) (end 112 137.5) (width 1) (layer "F.Cu") (net 2))
+  (segment (start 81.28 137.16) (end 89.849966 145.729966) (width 1) (layer "B.Cu") (net 1))
+  (segment (start 112 127.24) (end 121.92 137.16) (width 1) (layer "F.Cu") (net 2))
   (segment (start 160.5 146.16) (end 160.5 156) (width 1) (layer "F.Cu") (net 2))
+  (segment (start 112 115.6) (end 112 127.24) (width 1) (layer "F.Cu") (net 2))
   (via (at 160.5 146.16) (size 2) (drill 0.4) (layers "F.Cu" "B.Cu") (net 2))
-  (via (at 112 137.5) (size 2) (drill 0.4) (layers "F.Cu" "B.Cu") (net 2))
+  (via (at 121.92 137.16) (size 2) (drill 0.4) (layers "F.Cu" "B.Cu") (net 2))
   (segment (start 161.66 145) (end 201.89 145) (width 1) (layer "B.Cu") (net 2))
-  (segment (start 116.74 142.24) (end 112 137.5) (width 1) (layer "B.Cu") (net 2))
-  (segment (start 160.5 146.16) (end 156.58 142.24) (width 1) (layer "B.Cu") (net 2))
+  (segment (start 121.92 137.16) (end 127 142.24) (width 1) (layer "B.Cu") (net 2))
+  (segment (start 156.58 142.24) (end 160.5 146.16) (width 1) (layer "B.Cu") (net 2))
+  (segment (start 127 142.24) (end 156.58 142.24) (width 1) (layer "B.Cu") (net 2))
   (segment (start 160.5 146.16) (end 161.66 145) (width 1) (layer "B.Cu") (net 2))
   (segment (start 204 147.11) (end 204 148.85) (width 1) (layer "B.Cu") (net 2))
   (segment (start 201.89 145) (end 204 147.11) (width 1) (layer "B.Cu") (net 2))
-  (segment (start 156.58 142.24) (end 116.74 142.24) (width 1) (layer "B.Cu") (net 2))
   (segment (start 210.5 147.11) (end 210.5 148.85) (width 1) (layer "F.Cu") (net 3))
   (segment (start 179 139) (end 174.5 143.5) (width 1) (layer "F.Cu") (net 3))
@@
   (segment (start 207 118.5) (end 207 136) (width 1) (layer "B.Cu") (net 6))
   (zone (net 6) (net_name "GND") (layers F&B.Cu) (hatch edge 0.508)
-    (connect_pads (clearance 2))
-    (min_thickness 2) (filled_areas_thickness no)
+    (connect_pads (clearance 1.5))
+    (min_thickness 1.5) (filled_areas_thickness no)
     (fill yes (thermal_gap 2) (thermal_bridge_width 2))
     (polygon
