File: docs/KiCad/Lunchbox_Sampler_Main_PCB/Lunchbox_Sampler_Main_PCB.kicad_pcb (KiCad board)
At the start: 2 copper layers, 198 x 85 mm, 31 parts, among them J1 Conn_01x14_MountingPin, J10 Conn_01x02, J11 NMJ4HCD2, J12 Conn_01x10, J13 Conn_01x08, J14 Conn_01x04, J16 NMJ4HCD2, J17 NMJ4HCD2, J18 NMJ4HCD2, J2 Conn_01x14_MountingPin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

Commit message: pcb updated
Parts:
- added J15: Conn_01x08, Connector_PinHeader_2.54mm:PinHeader_1x08_P2.54mm_Vertical, F.Cu at (76.6, 88.9)
- J14: value Conn_01x04 -> Conn_01x06; footprint Connector_PinHeader_2.54mm:PinHeader_1x04_P2.54mm_Vertical -> Connector_PinHeader_2.54mm:PinHeader_1x06_P2.54mm_Vertical
- moved J14 2.55 mm to (25.8, 98.0)
- moved J2 1.59 mm to (19.0, 89.0)
- moved J1 0.90 mm to (52.0, 45.7)
Routing:
- net GND: track 84.4 -> 86.6 mm
- net Net-(J2-Pad9): track 11.1 -> 12.7 mm
- net Net-(J2-Pad7): track 11.1 -> 12.7 mm
- net Net-(J2-Pad5): track 11.1 -> 12.7 mm
- net Net-(J2-Pad8): track 11.1 -> 12.7 mm
- net Net-(J2-Pad6): track 11.1 -> 12.7 mm
- net Net-(J2-Pad4): track 11.1 -> 12.7 mm
- net Net-(J2-Pad3): track 11.1 -> 12.7 mm
- net Net-(J2-Pad2): track 11.1 -> 12.7 mm
- net Net-(J2-Pad11): track 11.1 -> 12.7 mm
- net Net-(J2-Pad10): track 11.1 -> 12.7 mm
- net Net-(J2-Pad1): track 11.1 -> 12.7 mm
- net Net-(C1-Pad1): track 189.3 -> 190.9 mm
- net Net-(J14-Pad1): track 321.4 -> 320.2 mm
- net Net-(J1-Pad8): track 14.4 -> 15.3 mm
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