File: docs/KiCad/Lunchbox_Sampler_Main_PCB/Lunchbox_Sampler_Main_PCB.kicad_sch (KiCad schematic)
At the start: 31 parts, among them J1 Conn_01x14_MountingPin, J10 Conn_01x02, J11 NMJ4HCD2, J12 Conn_01x10, J13 Conn_01x08, J14 Conn_01x04, J16 NMJ4HCD2, J17 NMJ4HCD2, J18 NMJ4HCD2, J2 Conn_01x14_MountingPin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

Commit message: pcb updated
Parts:
- removed J14: Conn_01x04, Connector_PinHeader_2.54mm:PinHeader_1x04_P2.54mm_Vertical, symbol Connector_Generic:Conn_01x04
- added J14: Conn_01x06, Connector_PinHeader_2.54mm:PinHeader_1x06_P2.54mm_Vertical, symbol Connector_Generic:Conn_01x06
- added J15: Conn_01x08, Connector_PinHeader_2.54mm:PinHeader_1x08_P2.54mm_Vertical, symbol Connector_Generic:Conn_01x08
Connections:
- net GND: now also J15.1 (Pin_1), J15.2 (Pin_2), J15.3 (Pin_3), J15.4 (Pin_4), J15.5 (Pin_5), J15.6 (Pin_6), J15.7 (Pin_7), J15.8 (Pin_8)
- net at J2.12 (Pin_12), J4.2, R6.1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: now also J14.1 (Pin_1), J14.2 (Pin_2), J14.3 (Pin_3), J14.4 (Pin_4), J14.5 (Pin_5), J14.6 (Pin_6)
Changed lines of the file:
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@@
   (junction (at 367.03 76.2) (diameter 0) (color 0 0 0 0)
   )
-  (junction (at 124.46 193.04) (diameter 0) (color 0 0 0 0)
+  (junction (at 124.46 198.12) (diameter 0) (color 0 0 0 0)
   )
   (junction (at 193.04 203.2) (diameter 0) (color 0 0 0 0)
@@
   (junction (at 266.7 147.32) (diameter 0) (color 0 0 0 0)
   )
-  (junction (at 124.46 190.5) (diameter 0) (color 0 0 0 0)
+  (junction (at 124.46 203.2) (diameter 0) (color 0 0 0 0)
   )
   (junction (at 364.49 19.05) (diameter 0) (color 0 0 0 0)
@@
   (junction (at 114.3 152.4) (diameter 0) (color 0 0 0 0)
   )
+  (junction (at 219.71 209.55) (diameter 0) (color 0 0 0 0)
+  )
   (junction (at 193.04 208.28) (diameter 0) (color 0 0 0 0)
   )
@@
   (junction (at 241.3 147.32) (diameter 0) (color 0 0 0 0)
   )
+  (junction (at 219.71 201.93) (diameter 0) (color 0 0 0 0)
+  )
   (junction (at 368.3 59.69) (diameter 0) (color 0 0 0 0)
   )
@@
   (junction (at 193.04 213.36) (diameter 0) (color 0 0 0 0)
   )
+  (junction (at 219.71 214.63) (diameter 0) (color 0 0 0 0)
+  )
+  (junction (at 219.71 196.85) (diameter 0) (color 0 0 0 0)
+  )
   (junction (at 292.1 142.24) (diameter 0) (color 0 0 0 0)
   )
   (junction (at 193.04 210.82) (diameter 0) (color 0 0 0 0)
   )
+  (junction (at 124.46 205.74) (diameter 0) (color 0 0 0 0)
+  )
+  (junction (at 219.71 204.47) (diameter 0) (color 0 0 0 0)
+  )
   (junction (at 243.84 144.78) (diameter 0) (color 0 0 0 0)
   )
+  (junction (at 219.71 199.39) (diameter 0) (color 0 0 0 0)
+  )
+  (junction (at 124.46 208.28) (diameter 0) (color 0 0 0 0)
+  )
+  (junction (at 219.71 212.09) (diameter 0) (color 0 0 0 0)
+  )
   (junction (at 193.04 205.74) (diameter 0) (color 0 0 0 0)
   )
   (junction (at 375.92 53.34) (diameter 0) (color 0 0 0 0)
   )
-  (junction (at 124.46 195.58) (diameter 0) (color 0 0 0 0)
+  (junction (at 219.71 207.01) (diameter 0) (color 0 0 0 0)
   )
   (junction (at 386.08 21.59) (diameter 0) (color 0 0 0 0)
   )
+  (junction (at 124.46 200.66) (diameter 0) (color 0 0 0 0)
+  )
   (junction (at 193.04 215.9) (diameter 0) (color 0 0 0 0)
   )
@@
     (stroke (width 0) (type default) (color 0 0 0 0))
   )
+  (wire (pts (xy 124.46 205.74) (xy 124.46 208.28))
+    (stroke (width 0) (type default) (color 0 0 0 0))
+  )
   (wire (pts (xy 314.96 91.44) (xy 309.88 91.44))
     (stroke (width 0) (type default) (color 0 0 0 0))
@@
     (stroke (width 0) (type default) (color 0 0 0 0))
   )
+  (wire (pts (xy 219.71 212.09) (xy 219.71 214.63))
+    (stroke (width 0) (type default) (color 0 0 0 0))
+  )
+  (wire (pts (xy 219.71 199.39) (xy 219.71 201.93))
+    (stroke (width 0) (type default) (color 0 0 0 0))
+  )
   (wire (pts (xy 265.43 77.47) (xy 171.45 77.47))
     (stroke (width 0) (type default) (color 0 0 0 0))
@@
     (stroke (width 0) (type default) (color 0 0 0 0))
   )
-  (wire (pts (xy 124.46 181.61) (xy 124.46 190.5))
+  (wire (pts (xy 124.46 181.61) (xy 124.46 198.12))
     (stroke (width 0) (type default) (color 0 0 0 0))
   )
@@
     (stroke (width 0) (type default) (color 0 0 0 0))
   )
-  (wire (pts (xy 124.46 190.5) (xy 124.46 193.04))
-    (stroke (width 0) (type default) (color 0 0 0 0))
-  )
   (wire (pts (xy 314.96 96.52) (xy 307.34 96.52))
     (stroke (width 0) (type default) (color 0 0 0 0))
@@
     (stroke (width 0) (type default) (color 0 0 0 0))
   )
-  (wire (pts (xy 124.46 193.04) (xy 124.46 195.58))
-    (stroke (width 0) (type default) (color 0 0 0 0))
-  )
   (wire (pts (xy 345.44 152.4) (xy 367.03 152.4))
     (stroke (width 0) (type default) (color 0 0 0 0))
@@
     (stroke (width 0) (type default) (color 0 0 0 0))
   )
+  (wire (pts (xy 219.71 214.63) (xy 219.71 218.44))
+    (stroke (width 0) (type default) (color 0 0 0 0))
+  )
   (wire (pts (xy 323.85 49.53) (xy 322.58 49.53))
     (stroke (width 0) (type default) (color 0 0 0 0))
@@
     (stroke (width 0) (type default) (color 0 0 0 0))
   )
+  (wire (pts (xy 124.46 208.28) (xy 124.46 210.82))
+    (stroke (width 0) (type default) (color 0 0 0 0))
+  )
   (wire (pts (xy 242.57 93.98) (xy 242.57 59.69))
     (stroke (width 0) (type default) (color 0 0 0 0))
@@
     (stroke (width 0) (type default) (color 0 0 0 0))
   )
+  (wire (pts (xy 124.46 200.66) (xy 124.46 203.2))
+    (stroke (width 0) (type default) (color 0 0 0 0))
+  )
   (wire (pts (xy 180.34 86.36) (xy 180.34 85.09))
     (stroke (width 0) (type default) (color 0 0 0 0))
   )
+  (wire (pts (xy 219.71 201.93) (xy 219.71 204.47))
+    (stroke (width 0) (type default) (color 0 0 0 0))
+  )
   (wire (pts (xy 322.58 44.45) (xy 322.58 31.75))
     (stroke (width 0) (type default) (color 0 0 0 0))
@@
     (stroke (width 0) (type default) (color 0 0 0 0))
   )
-  (wire (pts (xy 219.71 195.58) (xy 219.71 218.44))
+  (wire (pts (xy 219.71 195.58) (xy 219.71 196.85))
     (stroke (width 0) (type default) (color 0 0 0 0))
   )
@@
     (stroke (width 0) (type default) (color 0 0 0 0))
   )
+  (wire (pts (xy 124.46 203.2) (xy 124.46 205.74))
+    (stroke (width 0) (type default) (color 0 0 0 0))
+  )
+  (wire (pts (xy 219.71 204.47) (xy 219.71 207.01))
+    (stroke (width 0) (type default) (color 0 0 0 0))
+  )
   (wire (pts (xy 189.23 27.94) (xy 252.73 27.94))
     (stroke (width 0) (type default) (color 0 0 0 0))
@@
     (stroke (width 0) (type default) (color 0 0 0 0))
   )
+  (wire (pts (xy 124.46 198.12) (xy 124.46 200.66))
+    (stroke (width 0) (type default) (color 0 0 0 0))
+  )
   (wire (pts (xy 176.53 137.16) (xy 180.34 137.16))
     (stroke (width 0) (type default) (color 0 0 0 0))
@@
     (stroke (width 0) (type default) (color 0 0 0 0))
   )
+  (wire (pts (xy 219.71 207.01) (xy 219.71 209.55))
+    (stroke (width 0) (type default) (color 0 0 0 0))
+  )
   (wire (pts (xy 257.81 67.31) (xy 163.83 67.31))
     (stroke (width 0) (type default) (color 0 0 0 0))
@@
     (stroke (width 0) (type default) (color 0 0 0 0))
   )
-  (wire (pts (xy 124.46 195.58) (xy 124.46 198.12))
+  (wire (pts (xy 219.71 196.85) (xy 219.71 199.39))
+    (stroke (width 0) (type default) (color 0 0 0 0))
+  )
+  (wire (pts (xy 219.71 209.55) (xy 219.71 212.09))
     (stroke (width 0) (type default) (color 0 0 0 0))
   )
@@
     (pin "3")
     (pin "4")
+  )
+  (symbol (lib_id "Connector_Generic:Conn_01x08") (at 224.79 204.47 0) (unit 1)
+    (in_bom yes) (on_board yes) (fields_autoplaced)
+    (property "Reference" "J15" (id 0) (at 227.33 204.4699 0)
+      (effects (font (size 1.27 1.27)) (justify left))
+    )
+    (property "Value" "Conn_01x08" (id 1) (at 227.33 207.0099 0)
+      (effects (font (size 1.27 1.27)) (justify left))
+    )
+    (property "Footprint" "Connector_PinHeader_2.54mm:PinHeader_1x08_P2.54mm_Vertical" (id 2) (at 224.79 204.47 0)
+      (effects (font (size 1.27 1.27)) hide)
+    )
+    (property "Datasheet" "~" (id 3) (at 224.79 204.47 0)
+      (effects (font (size 1.27 1.27)) hide)
+    )
+    (pin "1")
+    (pin "2")
+    (pin "3")
+    (pin "4")
+    (pin "5")
+    (pin "6")
+    (pin "7")
+    (pin "8")
   )
   (symbol (lib_id "Connector_Generic:Conn_01x08") (at 267.97 35.56 0) (unit 1)
@@
     (pin "2")
   )
+  (symbol (lib_id "Connector_Generic:Conn_01x06") (at 129.54 203.2 0) (unit 1)
+    (in_bom yes) (on_board yes) (fields_autoplaced)
+    (property "Reference" "J14" (id 0) (at 132.08 203.1999 0)
+      (effects (font (size 1.27 1.27)) (justify left))
+    )
+    (property "Value" "Conn_01x06" (id 1) (at 132.08 205.7399 0)
+      (effects (font (size 1.27 1.27)) (justify left))
+    )
+    (property "Footprint" "Connector_PinHeader_2.54mm:PinHeader_1x06_P2.54mm_Vertical" (id 2) (at 129.54 203.2 0)
+      (effects (font (size 1.27 1.27)) hide)
+    )
+    (property "Datasheet" "~" (id 3) (at 129.54 203.2 0)
+      (effects (font (size 1.27 1.27)) hide)
+    )
+    (pin "1")
+    (pin "2")
+    (pin "3")
+    (pin "4")
+    (pin "5")
+    (pin "6")
+  )
   (symbol (lib_id "Mechanical:MountingHole") (at 92.3843 47.9212 0) (unit 1)
     (in_bom yes) (on_board yes) (fields_autoplaced)
@@
       (effects (font (size 1.27 1.27)) hide)
     )
-  )
-  (symbol (lib_id "Connector_Generic:Conn_01x04") (at 129.54 193.04 0) (unit 1)
-    (in_bom yes) (on_board yes) (fields_autoplaced)
-    (property "Reference" "J14" (id 0) (at 132.08 193.0399 0)
-      (effects (font (size 1.27 1.27)) (justify left))
-    )
-    (property "Value" "Conn_01x04" (id 1) (at 132.08 195.5799 0)
-      (effects (font (size 1.27 1.27)) (justify left))
-    )
-    (property "Footprint" "Connector_PinHeader_2.54mm:PinHeader_1x04_P2.54mm_Vertical" (id 2) (at 129.54 193.04 0)
-      (effects (font (size 1.27 1.27)) hide)
-    )
-    (property "Datasheet" "~" (id 3) (at 129.54 193.04 0)
-      (effects (font (size 1.27 1.27)) hide)
-    )
-    (pin "1")
-    (pin "2")
-    (pin "3")
-    (pin "4")
   )
   (symbol (lib_id "SamacSys_Parts:NMJ4HCD2") (at 246.38 16.51 0) (unit 1)
@@
       (reference "J13") (unit 1) (value "Conn_01x08") (footprint "Connector_PinHeader_2.54mm:PinHeader_1x08_P2.54mm_Vertical")
     )
-    (path "/72b67604-32e9-4311-9b3f-08f6da62bf33"
-      (reference "J14") (unit 1) (value "Conn_01x04") (footprint "Connector_PinHeader_2.54mm:PinHeader_1x04_P2.54mm_Vertical")
+    (path "/6c71e717-5ab8-4af0-9881-e9aeb7ccdec0"
+      (reference "J14") (unit 1) (value "Conn_01x06") (footprint "Connector_PinHeader_2.54mm:PinHeader_1x06_P2.54mm_Vertical")
+    )
+    (path "/117e65eb-cc29-4120-a414-a55cba034aa5"
+      (reference "J15") (unit 1) (value "Conn_01x08") (footprint "Connector_PinHeader_2.54mm:PinHeader_1x08_P2.54mm_Vertical")
     )
     (path "/04aff7d4-859c-4726-a9ca-ce94183e2a11"
